Commit message: Setup obstacles and grasping objects in gazebo

File: kortex_description/grippers/robotiq_2f_85/urdf/robotiq_2f_85_transmission_macro.xacro (robot description, xacro)
@@ -53,8 +53,8 @@
                 <hasPID/>
             </plugin>
-            <plugin name="gazebo_grasp_fix" filename="libgazebo_grasp_fix.so">
+            <!--<plugin name="gazebo_grasp_fix" filename="libgazebo_grasp_fix.so">
                 <arm>
                     <arm_name>my_robotiq_gripper</arm_name>
-                    <palm_link>${prefix}bracelet_link</palm_link> <!-- Gazebo merges links connected by fixed joints, so here we would have put gripper_base_link but it is merged with Bracelet_Link internally -->
+                    <palm_link>${prefix}bracelet_link</palm_link> --><!-- Gazebo merges links connected by fixed joints, so here we would have put gripper_base_link but it is merged with Bracelet_Link internally --><!--
                     <gripper_link> ${prefix}left_inner_finger </gripper_link>
                     <gripper_link> ${prefix}right_inner_finger </gripper_link>
@@ -67,6 +67,18 @@
                 <disable_collisions_on_attach>false</disable_collisions_on_attach>
                 <contact_topic>__default_topic__</contact_topic>
-            </plugin>
+            </plugin>-->
         </gazebo>
+      <gazebo reference="${prefix}left_inner_finger">
+        <mu1>100.0</mu1>
+        <mu2>100.0</mu2>
+        <minDepth>0.003</minDepth>
+        <maxVel>0</maxVel>
+      </gazebo>
+      <gazebo reference="${prefix}right_inner_finger">
+        <mu1>100.0</mu1>
+        <mu2>100.0</mu2>
+        <minDepth>0.003</minDepth>
+        <maxVel>0</maxVel>
+      </gazebo>
     </xacro:macro>
 </robot>

File: kortex_move_it_config/gen3_move_it_config/config/6dof/gen3.srdf.xacro (robot description, xacro)
@@ -23,5 +23,5 @@
     <!--GROUP STATES: Purpose: Define a named state for a particular group, in terms of joint values. This is useful to define states like 'folded arms'-->
     <group_state name="home" group="arm">
-        <joint name="$(arg prefix)joint_1" value="0" />
+        <joint name="$(arg prefix)joint_1" value="1.57" />
         <joint name="$(arg prefix)joint_2" value="0.26" />
         <joint name="$(arg prefix)joint_3" value="-2.27" />
@@ -31,5 +31,5 @@
     </group_state>
     <group_state name="retract" group="arm">
-        <joint name="$(arg prefix)joint_1" value="0" />
+        <joint name="$(arg prefix)joint_1" value="1.57" />
         <joint name="$(arg prefix)joint_2" value="-0.35" />
         <joint name="$(arg prefix)joint_3" value="-2.54" />

File: kortex_move_it_config/gen3_move_it_config/config/7dof/gen3.srdf.xacro (robot description, xacro)
@@ -24,5 +24,5 @@
     <!--GROUP STATES: Purpose: Define a named state for a particular group, in terms of joint values. This is useful to define states like 'folded arms'-->
     <group_state name="home" group="arm">
-        <joint name="$(arg prefix)joint_1" value="0" />
+        <joint name="$(arg prefix)joint_1" value="1.57" />
         <joint name="$(arg prefix)joint_2" value="0.26" />
         <joint name="$(arg prefix)joint_3" value="3.14" />
@@ -33,5 +33,5 @@
     </group_state>
     <group_state name="retract" group="arm">
-        <joint name="$(arg prefix)joint_1" value="0" />
+        <joint name="$(arg prefix)joint_1" value="1.57" />
         <joint name="$(arg prefix)joint_2" value="-0.35" />
         <joint name="$(arg prefix)joint_3" value="3.14" />

File: kortex_move_it_config/gen3_robotiq_2f_85_move_it_config/config/6dof/gen3_robotiq_2f_85.srdf.xacro (robot description, xacro)
@@ -36,5 +36,5 @@
     <!--GROUP STATES: Purpose: Define a named state for a particular group, in terms of joint values. This is useful to define states like 'folded arms'-->
     <group_state name="home" group="arm">
-        <joint name="$(arg prefix)joint_1" value="0" />
+        <joint name="$(arg prefix)joint_1" value="1.57" />
         <joint name="$(arg prefix)joint_2" value="0.26" />
         <joint name="$(arg prefix)joint_3" value="-2.27" />
@@ -44,5 +44,5 @@
     </group_state>
     <group_state name="retract" group="arm">
-        <joint name="$(arg prefix)joint_1" value="0" />
+        <joint name="$(arg prefix)joint_1" value="1.57" />
         <joint name="$(arg prefix)joint_2" value="-0.35" />
         <joint name="$(arg prefix)joint_3" value="-2.54" />

File: kortex_move_it_config/gen3_robotiq_2f_85_move_it_config/config/7dof/gen3_robotiq_2f_85.srdf.xacro (robot description, xacro)
@@ -37,5 +37,5 @@
     <!--GROUP STATES: Purpose: Define a named state for a particular group, in terms of joint values. This is useful to define states like 'folded arms'-->
     <group_state name="home" group="arm">
-        <joint name="$(arg prefix)joint_1" value="0" />
+        <joint name="$(arg prefix)joint_1" value="1.57" />
         <joint name="$(arg prefix)joint_2" value="0.26" />
         <joint name="$(arg prefix)joint_3" value="3.14" />
